Commit message: Console de régie web : refonte UI, retour caméra MJPEG, pilotage cmd_vel_web (SIM-ONLY)
Lot W3 partie sim du plan docs/etude-interface-web.md, sur demande : « retour
caméra + partie pilotage, un site agréable, pas une liste de boutons ».

Chaîne roues (contrat gelé, étendu) :
- twist_mux.yaml : entrée web (cmd_vel_web, prio 50) entre remote (100) et
  anim (10) — la télécommande physique garde structurellement la main
- test_twist_mux_contract.py : le contrat de priorités est désormais testé

Pilotage (SÉCURITÉ, sim uniquement) :
- message WS "drive" (x/z normalisés) : clamp silencieux [-1,1], refus
  NaN/inf/bool, canal séparé de la whitelist cmd
- drive_to_twist = plafond DUR côté backend (0,5 m/s / 1,0 rad/s défaut),
  re-clampé au dernier calcul avant publication
- drive_enabled défaut FALSE : le publisher cmd_vel_web n'est pas créé sans
  lui (aucune ligne ne PEUT publier de mouvement) ; WEB_DRIVE=true en sim
- DriveFlow pur (horloge injectée) : UN zéro 300 ms après la dernière
  consigne ; zéro immédiat sur déconnexion writer / timeout heartbeat /
  take_control / STOP
- vérifié e2e dans le conteneur : 16 Twist en salve 15 Hz, zéro unique à
  l'arrêt, consigne hors bornes (5.0) ressortie au plafond 0,5 m/s, lecteur
  refusé, 0,25 m/s observé jusqu'à /cmd_vel (mux + deadman traversés)

Retour caméra :
- capteur caméra gz ajouté à l'URDF (camera_link, 640x480@15) + système
  Sensors dans stage.sdf + bridge camera/image_raw
- endpoint GET /video : MJPEG multipart, encodage PIL JPEG q70 throttlé
  AVANT encodage (video_fps=10), 503 si flux tari > 2 s
- vérifié : frames JFIF réelles servies depuis la caméra du robot simulé

UI console (toujours vanilla, zéro CDN) :
- layout 2 colonnes : DIRECT sticky (vidéo, pad tactile/souris, manette
  Gamepad API deadzone 0.15, slider vitesse, readout lin/ang, STOP) et
  CONTENUS (recherche live, sections en cartes, mires calib* déplacées dans
  Technique > Calibration)
- pad grisé avec explication si drive_enabled=false ; émission 15 Hz gatée
  par écriture + zéro au relâchement

Tests 511 -> 540 verts. Docs : interfaces.md (drive, /video, hello étendu,
cmd_vel_web), operations.md (procédure conduite sim, rappel SIM-ONLY),
etude-interface-web.md §6, CLAUDE.md.

Implémentation : agent Opus sur spec fermée (chemin roues) ; revue + vérif
e2e Docker : session Fable. Le passage au vrai robot reste conditionné au
test scénique au sol puis au protocole caméra (plan §6, W3).

Co-Authored-By: Claude Fable 5 <noreply@anthropic.com>

File: conf/ros2_dependencies/robot_description/urdf/dadou_robot_gz.urdf.xacro (robot description, xacro)
@@ -29,4 +29,52 @@
   <gazebo reference="mouth_leds_joint">
     <preserveFixedJoint>true</preserveFixedJoint>
+  </gazebo>
+  <!-- ======== Caméra embarquée (SIM-ONLY, retour vidéo du pont web W3) ========
+       Petit link fixe à l'avant de la tête (tambour neck), regardant vers +x
+       (l'avant du robot) : la caméra suit donc le regard du cou, comme le fera
+       la webcam vision sur le vrai robot. preserveFixedJoint pour que camera_link
+       ne soit PAS fusionné dans head_link à la conversion URDF vers SDF (même
+       piège que les LED) ; sinon la référence gazebo du capteur ne trouverait
+       plus son link et la caméra ne serait pas montée. -->
+  <link name="camera_link">
+    <visual>
+      <geometry><box size="0.03 0.05 0.03"/></geometry>
+      <material name="black"/>
+    </visual>
+    <xacro:box_inertial m="0.05" x="0.03" y="0.05" z="0.03"/>
+  </link>
+  <joint name="camera_joint" type="fixed">
+    <parent link="head_link"/>
+    <child link="camera_link"/>
+    <!-- Devant la tête (rayon du tambour + demi-épaisseur), à mi-hauteur. -->
+    <origin xyz="${head_radius + 0.015} 0 ${head_height/2}"/>
+  </joint>
+  <gazebo reference="camera_joint">
+    <preserveFixedJoint>true</preserveFixedJoint>
+  </gazebo>
+  <!-- Capteur caméra gz. La caméra gz regarde le long de +x du link : orientée
+       vers l'avant sans rotation. <topic> EXPLICITE (camera/image_raw) pour ne
+       PAS dépendre du nom auto-généré scoppé sur le monde/modèle
+       (/world/stage/model/.../sensor/.../image) ; le bridge (gz_bridge.yaml)
+       s'y abonne tel quel. NB : le rendu caméra exige le système gz Sensors,
+       ajouté au monde stage.sdf (sans lui, aucune image n'est publiée). -->
+  <gazebo reference="camera_link">
+    <sensor name="camera" type="camera">
+      <camera>
+        <horizontal_fov>1.047</horizontal_fov>
+        <image>
+          <width>640</width>
+          <height>480</height>
+          <format>R8G8B8</format>
+        </image>
+        <clip>
+          <near>0.1</near>
+          <far>100.0</far>
+        </clip>
+      </camera>
+      <always_on>1</always_on>
+      <update_rate>15</update_rate>
+      <topic>camera/image_raw</topic>
+    </sensor>
   </gazebo>
   <!-- Roue folle : elle est modélisée en sphère fixe, elle doit glisser. -->
