Commit message: Sim : visualisation des LED par matériaux émissifs Gazebo (corps, bouche, yeux)
Les LED du robot (ruban corps 513-673, bouche-matrice, yeux) n'existaient pas
en simulation. Cette visualisation est une APPROXIMATION assumée (repère visuel,
pas une réplique du rendu Adafruit) — l'avertissement est en tête de
robot_sim_lib/leds_logic.py.

Mécanisme (validé empiriquement sur la sim avant implémentation) :
- Le monde `stage` charge le système gz UserCommands qui expose
  /world/stage/material_color (gz.msgs.MaterialColor) : publier dessus change
  en runtime le matériau (diffuse/emissive) d'un visual nommé.
- Le bridge ros_gz de Jazzy convertit nativement
  ros_gz_interfaces/MaterialColor <-> gz.msgs.MaterialColor (paire vérifiée
  dans le binaire parameter_bridge). Zéro code C++, zéro plugin custom.

Contenu :
- URDF : liens body_leds_link + mouth_leds_link (boîtes fines émissives sur la
  face avant du torse, joints fixes, sans collision, masse 0.05 kg). PIÈGE
  contourné : la conversion URDF->SDF « lumpe » les liens à joint fixe dans le
  parent (nom de visual imprévisible) → preserveFixedJoint dans
  dadou_robot_gz.urdf.xacro. Vérifié sur le SDF généré (gz sdf -p) :
  body_leds_link_visual et mouth_leds_link_visual sont des visuals distincts.
  Les yeux réutilisent left/right_eye_link_visual (joints mobiles, déjà stables).
- robot_sim/scripts/leds_sim_node (package AUTONOME, aucun import robot.* ni
  dadou_utils_ros, même règle que robot_drive) : s'abonne à robot_lights et
  face (StringTime), résout les séquences via les MÊMES json que le vrai robot
  (robot_lights.json / lights_base.json / colors.json, montés dans le conteneur),
  publie /material_color à 10 Hz. Anti-spam : ne publie que si la couleur change
  (MaterialColor est une commande UserCommands, pas un flux), sauf effets animés.
  Horloge ROS (sim_time), jamais time.time().
- robot_sim_lib/leds_logic.py : logique pure (timeline des briques, effets
  approximés — blink créneau 1 Hz, pulse sinus, sparkle RNG seedé par pas de
  temps, rainbow/color_cycle cycle HSV), temps toujours injecté → testable.
  Face : approximation V1 (expressions = bitmaps, pas de mapping couleur juste) :
  toute expression allume bouche GOLD + yeux AQUA, stop éteint.
- Bridge /material_color -> /world/stage/material_color (ROS_TO_GZ), node ajouté
  au sim.launch.py, json/ copié dans l'image + monté en volume (itération sans
  rebuild).
- 21 tests unitaires host (robot/tests/unit/test_leds_logic.py) : timeline,
  bornes, loop, stop, brightness, effets déterministes. 162 tests verts au total
  (141 préexistants dont gaze_follower commité en parallèle + 21 nouveaux).

Divergences assumées vs robot/actions/lights.py (documentées dans le code) :
- timeline « naturelle » (segment i = fin du précédent → position_i × durée),
  sans répliquer le calcul particulier du premier élément de Sequence ;
- stop/fin de séquence → éteint (pas de retour à une séquence par défaut).

Vérifié par agent dans un conteneur jetable isolé (ROS_DOMAIN_ID=99, jamais 42) :
build colcon OK, node démarre, "devil"→rouge, "stop"→noir, effet animé republie
à chaque tick, séquence inconnue → erreur logguée sans crash, face "happy" →
bouche GOLD + yeux AQUA. Reste à faire : vérification visuelle GUI (l'URDF
spawné doit être rechargé → redémarrer le conteneur sim).

Implémentation : Agent Sonnet sur spec fermée (session Fable). Revue : Fable.

Co-Authored-By: Claude Opus 4.8 (1M context) <noreply@anthropic.com>

File: conf/ros2_dependencies/robot_description/urdf/dadou_robot.urdf.xacro (robot description, xacro)
@@ -44,4 +44,16 @@
   <xacro:property name="eye_offset_y" value="0.18"/>
   <xacro:property name="eye_offset_z" value="0.28"/>
+  <!-- Ruban LED "corps" (zone 513-673 du ruban physique) : boîte fine plaquée
+       sur la face avant du torse, ~80% de la hauteur, ~60% de la largeur. -->
+  <xacro:property name="body_leds_height" value="${0.8*torso_height}"/>
+  <xacro:property name="body_leds_width" value="${0.6*torso_width}"/>
+  <xacro:property name="body_leds_thickness" value="0.01"/>
+  <xacro:property name="body_leds_mass" value="0.05"/>
+  <!-- Matrice LED "bouche" (LED 0-384) : petite boîte en haut de la face avant,
+       au-dessus du ruban corps. -->
+  <xacro:property name="mouth_leds_width" value="0.12"/>
+  <xacro:property name="mouth_leds_height" value="0.08"/>
+  <xacro:property name="mouth_leds_thickness" value="0.01"/>
+  <xacro:property name="mouth_leds_mass" value="0.05"/>
   <!-- Course des servos : 0..180° matériel, centrée dans le modèle -->
   <xacro:property name="servo_lower" value="${-pi/2}"/>
@@ -52,4 +64,7 @@
   <material name="grey"><color rgba="0.55 0.55 0.55 1"/></material>
   <material name="blue_drum"><color rgba="0.15 0.20 0.35 1"/></material>
+  <!-- LED éteintes par défaut (couleur réelle pilotée en runtime par leds_sim_node
+       en sim, via matériaux émissifs gz ; sur le vrai robot ce sont des NeoPixel). -->
+  <material name="leds_off"><color rgba="0.05 0.05 0.05 1"/></material>
   <!-- ======== Macros d'inertie ======== -->
   <xacro:macro name="box_inertial" params="m x y z">
@@ -207,3 +222,33 @@
   <xacro:eye side="left" y_sign="1"/>
   <xacro:eye side="right" y_sign="-1"/>
+  <!-- ======== LED : visualisation des rubans réels (couleur pilotée en runtime) ========
+       Purement visuel : pas de <collision>, masse négligeable, joints FIXES sur le
+       torse. Le +x est la face avant (cf. disposition roues/caisson ci-dessus). -->
+  <!-- Ruban "corps" : de la base du torse jusqu'à 80% de sa hauteur. -->
+  <link name="body_leds_link">
+    <visual>
+      <geometry><box size="${body_leds_thickness} ${body_leds_width} ${body_leds_height}"/></geometry>
+      <material name="leds_off"/>
+    </visual>
+    <xacro:box_inertial m="${body_leds_mass}" x="${body_leds_thickness}" y="${body_leds_width}" z="${body_leds_height}"/>
+  </link>
+  <joint name="body_leds_joint" type="fixed">
+    <parent link="torso_link"/>
+    <child link="body_leds_link"/>
+    <origin xyz="${torso_length/2 + body_leds_thickness/2} 0 ${0.4*torso_height}"/>
+  </joint>
+  <!-- Matrice "bouche" : au-dessus du ruban corps, avec une marge sous le sommet
+       du torse pour ne pas chevaucher visuellement les deux zones. -->
+  <link name="mouth_leds_link">
+    <visual>
+      <geometry><box size="${mouth_leds_thickness} ${mouth_leds_width} ${mouth_leds_height}"/></geometry>
+      <material name="leds_off"/>
+    </visual>
+    <xacro:box_inertial m="${mouth_leds_mass}" x="${mouth_leds_thickness}" y="${mouth_leds_width}" z="${mouth_leds_height}"/>
+  </link>
+  <joint name="mouth_leds_joint" type="fixed">
+    <parent link="torso_link"/>
+    <child link="mouth_leds_link"/>
+    <origin xyz="${torso_length/2 + mouth_leds_thickness/2} 0 ${0.9*torso_height}"/>
+  </joint>
 </robot>

File: conf/ros2_dependencies/robot_description/urdf/dadou_robot_gz.urdf.xacro (robot description, xacro)
@@ -18,4 +18,16 @@
 <robot xmlns:xacro="http://www.ros.org/wiki/xacro" name="dadou_robot">
   <xacro:include filename="dadou_robot.urdf.xacro"/>
+  <!-- LED : joints fixes qu'il ne faut PAS laisser "lumper" par la conversion
+       URDF->SDF (sinon leurs visuals fusionnent dans le lien parent, avec un nom
+       du style "base_link_fixed_joint_lump__torso_link_visual_2" imprévisible).
+       preserveFixedJoint garde body_leds_link_visual / mouth_leds_link_visual
+       comme visuals distincts, avec un nom stable pour le bridge MaterialColor
+       (voir robot_sim/robot_sim_lib/leds_logic.py + config/gz_bridge.yaml). -->
+  <gazebo reference="body_leds_joint">
+    <preserveFixedJoint>true</preserveFixedJoint>
+  </gazebo>
+  <gazebo reference="mouth_leds_joint">
+    <preserveFixedJoint>true</preserveFixedJoint>
+  </gazebo>
   <!-- Roue folle : elle est modélisée en sphère fixe, elle doit glisser. -->
   <gazebo reference="caster_rear_link">
