Commit message: Sim : le modèle de Didier redessiné d'après les photos (visuel seul, physique intacte)
Le modèle de simulation ne ressemblait pas au robot : cylindre bleu pour la tête,
deux sphères grises pour les yeux, deux tiges rondes pour les bras. Relecture des
photos (docs/pictures/bout-small.jpeg vue de scène, mouth.jpg tête+yeux de près,
wheel-motor.jpg base et roues, duvam.net/didier vues avant/arrière) et refonte de
la silhouette :

- base : caisse de tôle larmée rouge cerclée d'acier noir, montants d'angle,
  roues cranelées DÉBORDANTES avec jante et pignon de chaîne, flèche arrière +
  chape portant la roue folle (dessinée en vraie roue pneumatique) ;
- torse : colonne de planches plus large que profonde, gros haut-parleur rond en
  façade (la bouche SONORE), deux ouïes à lamelles, mât d'acier à l'arrière,
  bossages d'épaule, arbre de cou visible ;
- tête : tambour clair à FACE AVANT PLANE (le vrai est un prisme hexagonal),
  chapeau bleu, portant la matrice LED du visage ;
- yeux : cloches type phare (cylindres étagés) au bout d'une ARCHE d'acier qui
  enjambe la tête, matrice LED en face avant ;
- bras : pales de bois plates, face large vers l'avant (elles balaient d'avant en
  arrière par la tranche, comme des rames).

Correction de fond au passage : la matrice LED « bouche » (0-384) était posée sur
le TORSE. Elle est sur la TÊTE — elle tourne donc désormais avec le cou, comme sur
le vrai robot. Les matrices des yeux (384-511) sont dessinées, ce qu'elles
n'étaient pas.

Contraintes de sûreté tenues : AUCUN changement de physique. Collisions, masses,
inerties, wheel_radius/wheel_separation et paramètres DiffDrive sont identiques au
modèle validé. Toute la décoration passe par des <visual> ajoutés dans les liens
existants (zéro masse, zéro collision). La roue folle reste une SPHÈRE glissante
en collision bien qu'elle soit dessinée en roue, et la caisse est DESSINÉE plus
étroite que sa collision (l'écart va dans le sens sûr : le robot simulé se cogne
plus tôt, jamais plus tard).

Conséquences côté sim :
- chaque zone LED a désormais son propre link protégé par preserveFixedJoint, y
  compris les yeux : leur link porte maintenant plusieurs visuals (la cloche), donc
  « le seul visual du link œil » n'était plus la matrice. leds_sim_node vise
  left/right_eye_leds_link_visual.
- la caméra embarquée passe sur le DESSUS de la tête : sa place réelle, et la face
  avant est désormais occupée par la matrice du visage. Elle ne sert qu'au retour
  vidéo web (le suivi de personne consomme /vision/person_box, pas cette image).

Vérifié : 443 tests verts ; géométrie contrôlée par rendu orthographique hors ligne
du xacro (z-buffer maison, joints à zéro), qui a révélé et fait corriger trois
défauts invisibles à la lecture du XML — plaque LED du visage enterrée dans le
tambour cylindrique (d'où la face plane ajoutée), pales de bras tournées de 90°,
et roues ne débordant pas de la caisse.

Co-Authored-By: Claude Opus 4.8 (1M context) <noreply@anthropic.com>

File: conf/ros2_dependencies/robot_description/urdf/dadou_robot_gz.urdf.xacro (robot description, xacro)
@@ -21,11 +21,20 @@
        URDF->SDF (sinon leurs visuals fusionnent dans le lien parent, avec un nom
        du style "base_link_fixed_joint_lump__torso_link_visual_2" imprévisible).
-       preserveFixedJoint garde body_leds_link_visual / mouth_leds_link_visual
-       comme visuals distincts, avec un nom stable pour le bridge MaterialColor
-       (voir robot_sim/robot_sim_lib/leds_logic.py + config/gz_bridge.yaml). -->
+       preserveFixedJoint garde <link>_visual comme visual distinct, avec un nom
+       stable pour le bridge MaterialColor (voir robot_sim/scripts/leds_sim_node
+       + config/gz_bridge.yaml).
+       Les yeux ont désormais une COQUE (cloche en cylindres étagés) en plus de
+       leur matrice : leur matrice a donc son propre link, comme le corps et la
+       bouche, au lieu de compter sur "le seul visual du link œil". -->
   <gazebo reference="body_leds_joint">
     <preserveFixedJoint>true</preserveFixedJoint>
   </gazebo>
   <gazebo reference="mouth_leds_joint">
+    <preserveFixedJoint>true</preserveFixedJoint>
+  </gazebo>
+  <gazebo reference="left_eye_leds_joint">
+    <preserveFixedJoint>true</preserveFixedJoint>
+  </gazebo>
+  <gazebo reference="right_eye_leds_joint">
     <preserveFixedJoint>true</preserveFixedJoint>
   </gazebo>
@@ -47,6 +56,11 @@
     <parent link="head_link"/>
     <child link="camera_link"/>
-    <!-- Devant la tête (rayon du tambour + demi-épaisseur), à mi-hauteur. -->
-    <origin xyz="${head_radius + 0.015} 0 ${head_height/2}"/>
+    <!-- SUR LE DESSUS de la tête, légèrement en avant : la face avant du tambour
+         est maintenant occupée par la matrice LED "bouche" (mouth_leds_link), et
+         c'est aussi là qu'est la vraie caméra du robot (posée sur la tête, cf.
+         validation du gaze du 2026-07-12). Elle regarde toujours vers +x et suit
+         donc le cou. Seul consommateur : le retour vidéo web — le suivi de
+         personne, lui, consomme /vision/person_box, pas cette image. -->
+    <origin xyz="${head_radius/2} 0 ${head_height + 0.025}"/>
   </joint>
   <gazebo reference="camera_joint">
